File: KiCad_Project/26_POWER(RK809-5)_1_PMIC.kicad_sch (KiCad schematic)
At the start: 82 parts, among them X2 32.768kHz

Commit message: Update additional PCBs
Add WIFI PCB to get best antenna
Add Display Debbugger to get interface pinout
Parts:
- removed C111, C116, C126: 1uF, Capacitor_SMD:C_0402_1005Metric, symbol LCSC Taish-easyedapro:CL05A105KP5NNNC
- removed R118, R124, R125, R126, R127, R38, R47, R74, R76: 0Ω, LCSC Taish-easyedapro:R0402, symbol LCSC Taish-easyedapro:ERJ2GE0R00X
- removed R41, R42, R43: 0402WGF1000TCE, LCSC Taish-easyedapro:R0402, symbol LCSC Taish-easyedapro:0402WGF1000TCE
Connections:
- net GND: now also U21.56 (BATDIV); no longer U111.47 (GNDREF), U111.62 (SNSP), U111.63 (SNSN), U111.69 (EPAD)
- net HPL_OUT: no longer U111.39 (HPL_OUT)
- net HPR_OUT: no longer U111.41 (HPR_OUT)
- net HP_SNS: no longer U111.40 (HP_SNS)
- net I2C0_SCL_PMIC: no longer U111.1 (SCL)
- net I2C0_SDA_PMIC: no longer U111.2 (SDA)
- net I2S1_LRCK_TX_M0_PMIC: no longer U111.14 (LRCLK)
- net I2S1_MCLK_M0_PMIC: no longer U111.16 (MCLK)
- net I2S1_SCLK_TX_M0_PMIC: no longer U111.15 (BCLK)
- net I2S1_SDI0_M0/PDM: no longer U111.18 (SDO/PDMDATA)
- net I2S1_SDO0_M0_PMIC: no longer U111.17 (SDI)
- net PDM_CLK0_M0_PMIC: no longer U111.19 (PDMCLK)
- net PMIC_INT_L: no longer U111.7 (INT)
- net PMIC_SLEEP_H: no longer U111.49 (SLEEP)
- net PWRON_KEY: no longer U111.52 (PWRON)
- net RESETN: no longer U111.67 (RESETB)
- net VCC3V3_PMU: no longer U111.31 (LDO6)
- net VCC3V3_SD: now also U21.58 (SWOUT2)
- net VCC3V3_SYS: now also U21.54 (VCC9), U21.57 (VCC8); no longer U111.10 (VCC2), U111.11 (VCC1), U111.22 (VCC5), U111.24 (VCC3), U111.30 (VCC6), U111.4 (VCC7), U111.66 (VCC4)
- net VCCA1V8_IMAGE: no longer U111.6 (LDO9)
- net VCCA1V8_PMU: no longer U111.5 (LDO8)
- net VCCA_1V8: no longer U111.3 (LDO7)
- net VCCIO_ACODEC: no longer U111.28 (LDO4)
- net VCCIO_SD: no longer U111.29 (LDO5)
- net VCC_3V3: now also U21.55 (SWOUT1)
- net VCC_DDR: no longer U111.26 (VBUCK3)
- net VDDA0V9_IMAGE: no longer U111.23 (LDO1)
- net VDDA0V9_PMU: no longer U111.20 (LDO3)
- net VDDA_0V9: no longer U111.21 (LDO2)
- net VDD_GPU: no longer U111.8 (FB2)
- net VDD_LOGIC: no longer U111.13 (FB1)
- net VDD_NPU: no longer U111.64 (FB4)
- net at C138.1, D26.3 (K), U21.45 (VCC_RTC): no longer U111.45 (VCC_RTC)
- net at C139.2, L8.2, U21.33 (VCC_SPK_HP): no longer U111.33 (VCC_SPK_HP)
- net at L3.2, U21.12 (SW1): no longer U111.12 (SW1)
- net at C137.2, U21.46 (VREF): no longer U111.46 (VREF)
- net at C140.2, U21.50 (XIN), X2.2: no longer U111.50 (XIN)
- net at C143.1, U21.51 (XOUT), X2.1: no longer U111.51 (XOUT)
- net at U111.56 (BAT1): no longer U21.56 (BATDIV)
- net at U111.60 (GATE): no longer U21.60 (EXT_EN)
- net at U111.61 (ADC/GPIO): no longer U21.61 (VDC)
- net at R50.2, U21.68 (CLK32K): no longer U111.68 (CLK32K)
- net at U111.55 (USB): no longer U21.55 (SWOUT1)
- net at C150.1, C152.2, U21.43 (MIC1p): no longer U111.43 (MIC1p)
- net at C151.2, R48.1, R51.2: now also U21.61 (VDC)
- net at L7.1, U21.53 (SW5): no longer U111.53 (SW5)
- net at C147.2, U21.44 (VCC_1P8A): no longer U111.44 (VCC_1P8A)
- net at L10.1, U21.32 (SPK_OUTp): no longer U111.32 (SPK_OUTp)
- net at L9.1, U21.34 (SPK_OUTn): no longer U111.34 (SPK_OUTn)
- net at C145.2, U21.35 (VCC_CPVSS): no longer U111.35 (VCC_CPVSS)
- net at C141.1, U21.36 (CPn): no longer U111.36 (CPn)
- net at C141.2, U21.37 (CPp): no longer U111.37 (CPp)
- net at C144.2, U21.38 (VCC_CPVDD): no longer U111.38 (VCC_CPVDD)
- net at U21.42 (MIC1n): no longer U111.42 (MIC1n)
- net at C146.2, U21.48 (VCC_1P8D): no longer U111.48 (VCC_1P8D)
- net at R46.1: now also U21.59 (FB5)
- net at R44.2, R45.2, U21.27 (FB3): no longer U111.27 (FB3)
- net at L6.1, U21.25 (SW3): no longer U111.25 (SW3)
- net at L4.1, U21.65 (SW4): no longer U111.65 (SW4)
- net at L5.2, U21.9 (SW2): no longer U111.9 (SW2)
- net at U111.54 (BOOST): no longer U21.54 (VCC9)
- net at U111.57 (VBAT2): no longer U21.57 (VCC8)
- net at U111.58 (SYS): no longer U21.58 (SWOUT2)
- net at U111.59 (SYS): no longer U21.59 (FB5)
Other:
- note removed: "P when 817"
- moved on the sheet: U111A, U111B, U111C, U111D
